File: AVI1861.kicad_pcb (KiCad board)
At the start: 2 copper layers, 29.9 x 17.2 mm, 9 parts, among them J1 1861, U1 LINE, U2 FRAME, U3 4021, U4 4040, U5 74LVC1G17, U6 74LVC2G07

Commit message: Revision B changes
Parts:
- C1, C2: value 0.1u -> 0.22u
- U3: value 4021 -> 4014
Connections:
- U1 pad 6: Net-(U1-Pad16) -> GND
- U1 pad 7: Net-(U1-Pad16) -> GND
- U1 pad 8: Net-(U1-Pad16) -> GND
- U1 pad 9: Net-(U1-Pad16) -> GND
- U3 pad 10: /~{CLK} -> Net-(U1-Pad16)
Routing:
- net /~{CLK}: track 47.5 -> 15.2 mm, vias 3 -> 1
- net Net-(U1-Pad16): track 7.68 -> 29.7 mm, vias 0 -> 2
- net VCC: track 58.0 -> 49.6 mm
- net GND: track 3.27 -> 9.11 mm
- net /~{COMP SYNC}: track 12.3 -> 13.0 mm
Other:
- board text added: "0.2"
- board text added: "Rev B"
- board text removed: "0.1"
- board text removed: "Rev A"
