File: AVI1861.kicad_sch (KiCad schematic)
At the start: 9 parts, among them J1 1861, U1 LINE, U2 FRAME, U3 4021, U4 4040, U5 74LVC1G17, U6 74LVC2G07

Commit message: Revision B changes
Parts:
- C1, C2: value 0.1u -> 0.22u
- U3: value 4021 -> 4014
Connections:
- net GND: now also U1.6 (I), U1.7 (I), U1.8 (I), U1.9 (I)
- net ~{CLK}: no longer U3.10 (CP)
- new net: U1.16 (I/O), U3.10 (CP)
Changed lines of the file:
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@@
   (junction (at 111.125 62.23) (diameter 0) (color 0 0 0 0)
   )
+  (junction (at 123.19 69.85) (diameter 0) (color 0 0 0 0)
+  )
+  (junction (at 95.885 84.455) (diameter 0) (color 0 0 0 0)
+  )
+  (junction (at 177.165 148.59) (diameter 0) (color 0 0 0 0)
+  )
+  (junction (at 161.29 120.65) (diameter 0) (color 0 0 0 0)
+  )
+  (junction (at 111.125 59.69) (diameter 0) (color 0 0 0 0)
+  )
   (junction (at 111.125 64.77) (diameter 0) (color 0 0 0 0)
-  )
-  (junction (at 123.19 69.85) (diameter 0) (color 0 0 0 0)
-  )
-  (junction (at 177.165 148.59) (diameter 0) (color 0 0 0 0)
-  )
-  (junction (at 161.29 120.65) (diameter 0) (color 0 0 0 0)
-  )
-  (junction (at 111.125 59.69) (diameter 0) (color 0 0 0 0)
-  )
-  (junction (at 133.35 67.31) (diameter 0) (color 0 0 0 0)
   )
   (junction (at 189.865 100.33) (diameter 0) (color 0 0 0 0)
@@
     (stroke (width 0) (type default) (color 0 0 0 0))
   )
-  (wire (pts (xy 111.125 92.71) (xy 111.125 64.77))
-    (stroke (width 0) (type default) (color 0 0 0 0))
-  )
   (wire (pts (xy 95.885 160.655) (xy 95.885 161.29))
     (stroke (width 0) (type default) (color 0 0 0 0))
@@
     (stroke (width 0) (type default) (color 0 0 0 0))
   )
+  (wire (pts (xy 95.885 84.455) (xy 111.125 84.455))
+    (stroke (width 0) (type default) (color 0 0 0 0))
+  )
   (wire (pts (xy 83.185 171.45) (xy 135.89 171.45))
     (stroke (width 0) (type default) (color 0 0 0 0))
@@
     (stroke (width 0) (type default) (color 0 0 0 0))
   )
+  (wire (pts (xy 200.66 92.71) (xy 200.66 107.95))
+    (stroke (width 0) (type default) (color 0 0 0 0))
+  )
   (wire (pts (xy 111.125 146.05) (xy 111.125 168.275))
     (stroke (width 0) (type default) (color 0 0 0 0))
@@
     (stroke (width 0) (type default) (color 0 0 0 0))
   )
-  (wire (pts (xy 81.915 92.71) (xy 111.125 92.71))
-    (stroke (width 0) (type default) (color 0 0 0 0))
-  )
   (wire (pts (xy 81.915 95.25) (xy 123.19 95.25))
     (stroke (width 0) (type default) (color 0 0 0 0))
@@
     (stroke (width 0) (type default) (color 0 0 0 0))
   )
-  (wire (pts (xy 200.025 67.31) (xy 200.025 107.95))
-    (stroke (width 0) (type default) (color 0 0 0 0))
-  )
   (wire (pts (xy 138.43 125.73) (xy 138.43 173.99))
     (stroke (width 0) (type default) (color 0 0 0 0))
@@
     (stroke (width 0) (type default) (color 0 0 0 0))
   )
+  (wire (pts (xy 200.66 107.95) (xy 205.74 107.95))
+    (stroke (width 0) (type default) (color 0 0 0 0))
+  )
   (wire (pts (xy 215.9 143.51) (xy 215.9 144.145))
     (stroke (width 0) (type default) (color 0 0 0 0))
@@
     (stroke (width 0) (type default) (color 0 0 0 0))
   )
+  (wire (pts (xy 81.915 92.71) (xy 200.66 92.71))
+    (stroke (width 0) (type default) (color 0 0 0 0))
+  )
   (wire (pts (xy 67.945 135.89) (xy 83.185 135.89))
     (stroke (width 0) (type default) (color 0 0 0 0))
@@
     (stroke (width 0) (type default) (color 0 0 0 0))
   )
-  (wire (pts (xy 200.025 67.31) (xy 133.35 67.31))
-    (stroke (width 0) (type default) (color 0 0 0 0))
-  )
   (wire (pts (xy 192.405 52.07) (xy 192.405 143.51))
     (stroke (width 0) (type default) (color 0 0 0 0))
@@
     (stroke (width 0) (type default) (color 0 0 0 0))
   )
-  (wire (pts (xy 200.025 107.95) (xy 205.74 107.95))
-    (stroke (width 0) (type default) (color 0 0 0 0))
-  )
   (wire (pts (xy 175.26 130.81) (xy 205.74 130.81))
     (stroke (width 0) (type default) (color 0 0 0 0))
@@
   )
   (wire (pts (xy 80.01 46.99) (xy 83.185 46.99))
+    (stroke (width 0) (type default) (color 0 0 0 0))
+  )
+  (wire (pts (xy 111.125 64.77) (xy 111.125 84.455))
     (stroke (width 0) (type default) (color 0 0 0 0))
   )
@@
       (effects (font (size 1.27 1.27)) (justify right))
     )
-    (property "Value" "0.1u" (id 1) (at 49.53 40.64 0)
+    (property "Value" "0.22u" (id 1) (at 49.53 40.64 0)
       (effects (font (size 1.27 1.27)) (justify right))
     )
@@
       (effects (font (size 1.27 1.27)) (justify left))
     )
-    (property "Value" "4021" (id 1) (at 217.9194 104.2471 0)
+    (property "Value" "4014" (id 1) (at 217.9194 104.2471 0)
       (effects (font (size 1.27 1.27)) (justify left))
     )
@@
       (effects (font (size 1.27 1.27)) (justify right))
     )
-    (property "Value" "0.1u" (id 1) (at 40.64 40.64 0)
+    (property "Value" "0.22u" (id 1) (at 40.64 40.64 0)
       (effects (font (size 1.27 1.27)) (justify right))
     )
@@
     )
     (path "/cd27d9d6-4b1c-41e1-930a-345e07318cb4"
-      (reference "C1") (unit 1) (value "0.1u") (footprint "Capacitor_SMD:C_0805_2012Metric")
+      (reference "C1") (unit 1) (value "0.22u") (footprint "Capacitor_SMD:C_0805_2012Metric")
     )
     (path "/0d451b2c-76c1-49b7-a4a3-fdfed6973363"
-      (reference "C2") (unit 1) (value "0.1u") (footprint "Capacitor_SMD:C_0805_2012Metric")
+      (reference "C2") (unit 1) (value "0.22u") (footprint "Capacitor_SMD:C_0805_2012Metric")
     )
     (path "/991900fa-e762-4315-8241-78bfda459a8f"
@@
     )
     (path "/bd315ccf-bb62-4d7b-b4e2-1c35cd575e8a"
-      (reference "U3") (unit 1) (value "4021") (footprint "AVI-1861-Reproduction:TSSOP-16_4.4x5.0mm_P0.65mm")
+      (reference "U3") (unit 1) (value "4014") (footprint "AVI-1861-Reproduction:TSSOP-16_4.4x5.0mm_P0.65mm")
     )
     (path "/60fb8c6c-3e51-4dc2-b64a-9b7c7559f0fb"

Commit message: Change 4040 to HC40404
Parts:
- U4: value 4040 -> HC4040
Changed lines of the file:
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@@
       (effects (font (size 1.27 1.27)) (justify left))
     )
-    (property "Value" "4040" (id 1) (at 57.2644 119.4871 0)
+    (property "Value" "HC4040" (id 1) (at 57.2644 119.4871 0)
       (effects (font (size 1.27 1.27)) (justify left))
     )
@@
     )
     (path "/60fb8c6c-3e51-4dc2-b64a-9b7c7559f0fb"
-      (reference "U4") (unit 1) (value "4040") (footprint "AVI-1861-Reproduction:TSSOP-16_4.4x5.0mm_P0.65mm")
+      (reference "U4") (unit 1) (value "HC4040") (footprint "AVI-1861-Reproduction:TSSOP-16_4.4x5.0mm_P0.65mm")
     )
     (path "/311ded7e-fb2d-4bc8-b096-fe14c1cdb651"
